File: Sheet2_LoRa.kicad_sch (KiCad schematic)
At the start: 4 parts, among them J2 CONSMA6.06, U3 Lambda62C-9S

Commit message: Fix: Applied footprint corrections and added missing libraries to tables
Parts:
- J2: footprint (none) -> FreedomUnit:CONSMA006.062
Changed lines of the file:
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@@
 			)
 		)
-		(property "Footprint" ""
+		(property "Footprint" "FreedomUnit:CONSMA006.062"
 			(at 148.59 55.88 0)
 			(effects
