File: Sheet4_USB.kicad_sch (KiCad schematic)
At the start: 4 parts, among them J3 USB4085-GF-A, U6 TPD2E001

Commit message: Fix: Applied footprint corrections and added missing libraries to tables
Parts:
- J3: footprint (none) -> Connector_USB:USB_C_Receptacle_GCT_USB4085
Changed lines of the file:
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@@
 			)
 		)
-		(property "Footprint" ""
+		(property "Footprint" "Connector_USB:USB_C_Receptacle_GCT_USB4085"
 			(at 80 90 0)
 			(effects
