File: Sheet3_Power.kicad_sch (KiCad schematic)
At the start: 19 parts, among them J1 Solar JST-PH, SW1 JS102011SAQN, U4 BQ25504, U5 MCP73831, U7 TPS7A02, U8 TPS22918

Commit message: Fix: Applied footprint corrections and added missing libraries to tables
Parts:
- BT1: footprint Connector_JST:JST_PH_S2B-PH-K_1x02_P2.00mm_Horizontal -> Battery:BatteryHolder_Keystone_1042_1x18650
- D1: footprint Resistor_SMD:R_0402_1005Metric -> Diode_SMD:D_SOD-323
- U5: footprint Connector_JST:JST_PH_S2B-PH-K_1x02_P2.00mm_Horizontal -> Package_TO_SOT_SMD:SOT-23-5
Changed lines of the file:
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@@
 			)
 		)
-		(property "Footprint" "Connector_JST:JST_PH_S2B-PH-K_1x02_P2.00mm_Horizontal"
+		(property "Footprint" "Battery:BatteryHolder_Keystone_1042_1x18650"
 			(at 165 55 0)
 			(effects
@@
 			)
 		)
-		(property "Footprint" "Resistor_SMD:R_0402_1005Metric"
+		(property "Footprint" "Diode_SMD:D_SOD-323"
 			(at 130 115 0)
 			(effects
@@
 			)
 		)
-		(property "Footprint" "Connector_JST:JST_PH_S2B-PH-K_1x02_P2.00mm_Horizontal"
+		(property "Footprint" "Package_TO_SOT_SMD:SOT-23-5"
 			(at 85 115 0)
 			(effects

Commit message: Fix: Comprehensive error resolution (nRF52840 pin remapping, footprint rebuilding)
Parts:
- U4: footprint Package_DFN_QFN:Texas_S-PVQFN-N16 -> Package_DFN_QFN:Texas_S-PVQFN-N16_EP2.7x2.7mm
Changed lines of the file:
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@@
 			)
 		)
-		(property "Footprint" "Package_DFN_QFN:Texas_S-PVQFN-N16"
+		(property "Footprint" "Package_DFN_QFN:Texas_S-PVQFN-N16_EP2.7x2.7mm"
 			(at 85 55 0)
 			(effects
