File: Sheet5_Peripherals.kicad_sch (KiCad schematic)
At the start: 26 parts, among them J4 Sharp LCD, J5 I2C Header, SW2 PTS636, SW3 PTS636, SW4 PTS636, SW5 PTS636, SW6 PTS636, SW7 PTS636, SW8 PTS636, U10 MX25R6435F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

Commit message: Fix: Applied footprint corrections and added missing libraries to tables
Parts:
- J4: footprint Capacitor_SMD:C_0402_1005Metric -> Connector_FFC-FPC:Hirose_FH12-10S-0.5SH_1x10-1MP_P0.50mm_Horizontal
- U9: footprint (none) -> RF_GPS:ublox_MAX
Changed lines of the file:
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@@
 			)
 		)
-		(property "Footprint" "Capacitor_SMD:C_0402_1005Metric"
+		(property "Footprint" "Connector_FFC-FPC:Hirose_FH12-10S-0.5SH_1x10-1MP_P0.50mm_Horizontal"
 			(at 175 55 0)
 			(effects
@@
 			)
 		)
-		(property "Footprint" ""
+		(property "Footprint" "RF_GPS:ublox_MAX"
 			(at 70 55 0)
 			(effects

Commit message: Fix: Comprehensive error resolution (nRF52840 pin remapping, footprint rebuilding)
Parts:
- SW2, SW3, SW4, SW5, SW6, SW7, SW8: footprint Button_Switch_SMD:SW_SPST_PTS636 -> FreedomUnit:SW_SPST_PTS636
Changed lines of the file:
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@@
 			)
 		)
-		(property "Footprint" "Button_Switch_SMD:SW_SPST_PTS636"
+		(property "Footprint" "FreedomUnit:SW_SPST_PTS636"
 			(at 215 150 0)
 			(effects
@@
 			)
 		)
-		(property "Footprint" "Button_Switch_SMD:SW_SPST_PTS636"
+		(property "Footprint" "FreedomUnit:SW_SPST_PTS636"
 			(at 273.65 110 0)
 			(effects
@@
 			)
 		)
-		(property "Footprint" "Button_Switch_SMD:SW_SPST_PTS636"
+		(property "Footprint" "FreedomUnit:SW_SPST_PTS636"
 			(at 75 150 0)
 			(effects
@@
 			)
 		)
-		(property "Footprint" "Button_Switch_SMD:SW_SPST_PTS636"
+		(property "Footprint" "FreedomUnit:SW_SPST_PTS636"
 			(at 250 150 0)
 			(effects
@@
 			)
 		)
-		(property "Footprint" "Button_Switch_SMD:SW_SPST_PTS636"
+		(property "Footprint" "FreedomUnit:SW_SPST_PTS636"
 			(at 280 75.32 0)
 			(effects
@@
 			)
 		)
-		(property "Footprint" "Button_Switch_SMD:SW_SPST_PTS636"
+		(property "Footprint" "FreedomUnit:SW_SPST_PTS636"
 			(at 180 150 0)
 			(effects
@@
 			)
 		)
-		(property "Footprint" "Button_Switch_SMD:SW_SPST_PTS636"
+		(property "Footprint" "FreedomUnit:SW_SPST_PTS636"
 			(at 40 150 0)
 			(effects
@@
 			)
 		)
-		(property "Footprint" "Button_Switch_SMD:SW_SPST_PTS636"
+		(property "Footprint" "FreedomUnit:SW_SPST_PTS636"
 			(at 112.62 33.65 0)
 			(effects
@@
 			)
 		)
-		(property "Footprint" "Button_Switch_SMD:SW_SPST_PTS636"
+		(property "Footprint" "FreedomUnit:SW_SPST_PTS636"
 			(at 145 150 0)
 			(effects
@@
 			)
 		)
-		(property "Footprint" "Button_Switch_SMD:SW_SPST_PTS636"
+		(property "Footprint" "FreedomUnit:SW_SPST_PTS636"
 			(at 110 150 0)
 			(effects
@@
 			)
 		)
-		(property "Footprint" "Button_Switch_SMD:SW_SPST_PTS636"
+		(property "Footprint" "FreedomUnit:SW_SPST_PTS636"
 			(at 150.08 171.35 0)
 			(effects
